File: circuit/_saved_verseWriter.sch (KiCad schematic (older format))
At the start: 40 parts, among them CON1 Micro_SD_Card, CON2 AVR-ISP-6, IC1 ATMEGA328P-A, P1 HOLE, P2 FT-232R, P4 SW, SW1 RESET, Y1 16M

Commit message: Add AVR-ISP
Parts:
- removed CON2: AVR-ISP-6, Pin_Headers:Pin_Header_Straight_2x03_Pitch2.54mm, symbol AVR-ISP-6
- added P5: AVR-ISP, Pin_Headers:Pin_Header_Straight_1x05_Pitch2.54mm, symbol CONN_01X05
- CON1: footprint SparkFun-Footprints:SF-MICRO-SD -> conn-io:HIROSE-MICROSD-DM3AT-SF
- P3: renamed from P?; footprint (none) -> Connectors_JST:JST_PH_B3B-PH-SM4-TB_03x2.00mm_Straight
Connections:
- net GND: now also P5.5 (P5)
- net at C4.1, IC1.29 ((PCINT14/~RESET~)PC6), R13.2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: now also P5.4 (P4)
- net at CON1.3 (CMD), IC1.15 ((PCINT3/OC2A/MOSI)PB3): now also P5.3 (P3)
- net at CON1.7 (DAT0), IC1.16 ((PCINT4/MISO)PB4): now also P5.1 (P1)
- net at CON1.5 (CLK), IC1.17 ((PCINT5/SCK)PB5): now also P5.2 (P2)
Changed lines of the file:
@@
 F 0 "CON1" H 7000 5350 50  0000 C CNN
 F 1 "Micro_SD_Card" H 8300 5350 50  0000 R CNN
-F 2 "SparkFun-Footprints:SF-MICRO-SD" H 8800 5050 50  0001 C CNN
+F 2 "conn-io:HIROSE-MICROSD-DM3AT-SF" H 8800 5050 50  0001 C CNN
 F 3 "" H 7650 4750 50  0000 C CNN
 	1    7650 4750
@@
 NoConn ~ 5650 5350
 $Comp
-L AVR-ISP-6 CON2
-U 1 1 58D7FAA6
-P 7400 6050
-F 0 "CON2" H 7295 6290 50  0000 C CNN
-F 1 "AVR-ISP-6" H 7135 5820 50  0000 L BNN
-F 2 "Pin_Headers:Pin_Header_Straight_2x03_Pitch2.54mm" V 6880 6090 50  0001 C CNN
-F 3 "" H 7375 6050 50  0000 C CNN
-	1    7400 6050
-	1    0    0    -1
-$EndComp
-$Comp
 L GND #PWR020
 U 1 1 58D83BBB
-P 7800 6150
-F 0 "#PWR020" H 7800 5900 50  0001 C CNN
-F 1 "GND" H 7800 6000 50  0000 C CNN
-F 2 "" H 7800 6150 60  0000 C CNN
-F 3 "" H 7800 6150 60  0000 C CNN
-	1    7800 6150
-	0    -1   -1   0
-$EndComp
-$Comp
-L VCC #PWR021
-U 1 1 58D83C16
-P 7800 5950
-F 0 "#PWR021" H 7800 5800 50  0001 C CNN
-F 1 "VCC" H 7800 6100 50  0000 C CNN
-F 2 "" H 7800 5950 50  0000 C CNN
-F 3 "" H 7800 5950 50  0000 C CNN
-	1    7800 5950
+P 7300 6150
+F 0 "#PWR020" H 7300 5900 50  0001 C CNN
+F 1 "GND" H 7300 6000 50  0000 C CNN
+F 2 "" H 7300 6150 60  0000 C CNN
+F 3 "" H 7300 6150 60  0000 C CNN
+	1    7300 6150
 	0    1    1    0
 $EndComp
 $Comp
-L CONN_01X03 P?
+L CONN_01X03 P3
 U 1 1 58D908C4
 P 5700 6650
-F 0 "P?" H 5700 6850 50  0000 C CNN
+F 0 "P3" H 5700 6850 50  0000 C CNN
 F 1 "IR" V 5800 6650 50  0000 C CNN
-F 2 "" H 5700 6650 50  0000 C CNN
+F 2 "Connectors_JST:JST_PH_B3B-PH-SM4-TB_03x2.00mm_Straight" H 5700 6650 50  0001 C CNN
 F 3 "" H 5700 6650 50  0000 C CNN
 	1    5700 6650
@@
 	4900 3350 5050 3350
 Wire Wire Line
-	5050 3350 5050 6150
+	5050 3350 5050 6050
 Wire Wire Line
 	8450 850  8750 850
@@
 Connection ~ 5050 5250
 Wire Wire Line
-	7250 5950 6300 5950
-Wire Wire Line
-	6300 5950 6300 5050
+	6300 5050 6300 5750
 Connection ~ 6300 5050
 Wire Wire Line
-	7250 6050 6150 6050
-Wire Wire Line
-	6150 6050 6150 4850
+	6150 4850 6150 5850
 Connection ~ 6150 4850
-Wire Wire Line
-	5050 6150 7250 6150
 Connection ~ 5050 5750
 Wire Wire Line
-	7500 6050 7950 6050
-Wire Wire Line
-	7950 6050 7950 5700
-Wire Wire Line
-	7950 5700 6400 5700
-Wire Wire Line
-	6400 5700 6400 4650
+	6400 4650 6400 5950
 Connection ~ 6400 4650
 Wire Wire Line
-	7800 5950 7500 5950
-Wire Wire Line
-	7800 6150 7500 6150
-Wire Wire Line
 	6150 1900 4900 1900
 Wire Wire Line
@@
 	4950 3150 4900 3150
 $Comp
-L VCC #PWR?
+L VCC #PWR021
 U 1 1 58D92722
 P 5350 6550
-F 0 "#PWR?" H 5350 6400 50  0001 C CNN
+F 0 "#PWR021" H 5350 6400 50  0001 C CNN
 F 1 "VCC" H 5350 6700 50  0000 C CNN
 F 2 "" H 5350 6550 50  0000 C CNN
@@
 $EndComp
 $Comp
-L GND #PWR?
+L GND #PWR022
 U 1 1 58D927B2
 P 5500 6650
-F 0 "#PWR?" H 5500 6400 50  0001 C CNN
+F 0 "#PWR022" H 5500 6400 50  0001 C CNN
 F 1 "GND" H 5500 6500 50  0000 C CNN
 F 2 "" H 5500 6650 60  0000 C CNN
@@
 Wire Wire Line
 	4950 6750 5500 6750
+$Comp
+L CONN_01X05 P5
+U 1 1 58D95536
+P 7500 5950
+F 0 "P5" H 7500 6250 50  0000 C CNN
+F 1 "AVR-ISP" V 7600 5950 50  0000 C CNN
+F 2 "Pin_Headers:Pin_Header_Straight_1x05_Pitch2.54mm" H 7500 5950 50  0001 C CNN
+F 3 "" H 7500 5950 50  0000 C CNN
+	1    7500 5950
+	1    0    0    -1
+$EndComp
+Wire Wire Line
+	6300 5750 7300 5750
+Wire Wire Line
+	6150 5850 7300 5850
+Wire Wire Line
+	6400 5950 7300 5950
+Wire Wire Line
+	5050 6050 7300 6050
 $EndSCHEMATC
