File: circuit/verseWriter.sch (KiCad schematic (older format))
At the start: 56 parts

Commit message: 配線変更
Parts:
- added C1: C, symbol C
- added P1: CONN_01X02, symbol CONN_01X02
- added P2: HOLE, symbol CONN_01X02
- added P3: Writer, symbol CONN_01X04
- D1, D10, D11, D12, D13, D14, D15, D16, D17, D18, D19, D2, D20, D21, D22, D23, D24, D3, D4, D5, D6, D7, D8, D9: renamed from D?; footprint (none) -> LEDs:LED_0805
- R1, R19, R2, R21, R4, R6, R9: renamed from R?; value R -> 1k; footprint (none) -> Resistors_SMD:R_0805_HandSoldering
- R10, R11, R12, R13, R14, R15, R16, R17: renamed from R?; footprint (none) -> Resistors_SMD:R_0805_HandSoldering
- R18, R20, R8: renamed from R?; value R -> 10; footprint (none) -> Resistors_SMD:R_0805_HandSoldering
- R3, R5, R7: renamed from R?; value R -> 2k; footprint (none) -> Resistors_SMD:R_0805_HandSoldering
- SW1: renamed from SW?; value SW_PUSH -> RESET
- gave numbers to parts that had none: 10
Connections:
- wire segments 180 -> 191
- no-connect marks 6 -> 9
Other:
- moved on the sheet: R2, R3, R4, R5, R6, R7

Commit message: internalBatteryType
Parts:
- removed C4: 0.1u, symbol C
- removed CON1: SD_Card, 10067847-001, symbol SD_Card
- removed D10, D11, D12, D13, D14, D15, D16, D17, D18, D19, D2, D20, D21, D22, D23, D24, D3, D4, D5, D6, D7, D8, D9: LED, LEDs:LED_0805, symbol LED
- removed IC1: ATMEGA328-P, DIL28, symbol ATMEGA328-P
- removed P1: CONN_01X02, symbol CONN_01X02
- removed P2: HOLE, symbol CONN_01X02
- removed Q1, Q2, Q3: c1815, symbol Q_NPN_BCE
- removed R13, R14, R15, R16, R17: 330, Resistors_SMD:R_0805_HandSoldering, symbol R
- removed R18, R20: 10, Resistors_SMD:R_0805_HandSoldering, symbol R
- removed R19, R21: 1k, Resistors_SMD:R_0805_HandSoldering, symbol R
- removed U1: LM2931Z-3.3/5.0, TO92-123, symbol LM2931Z-3.3/5.0
- added BT1, BT2: AAA, .pretty:AAA, symbol Battery_Cell
- added CON1: Micro_SD_Card, symbol Micro_SD_Card
- added D10, D11, D12, D2, D3, D4, D5, D6, D7, D8, D9: LED, LEDs:LED_0805, symbol LED-RESCUE-verseWriter
- added IC1: ATMEGA328P-A, Housings_QFP:TQFP-32_7x7mm_Pitch0.8mm, symbol ATMEGA328P-A
- added P1: HOLE, Pin_Headers:Pin_Header_Straight_1x03_Pitch2.54mm, symbol CONN_01X03
- added P4: SW, Pin_Headers:Pin_Header_Straight_1x03_Pitch2.54mm, symbol CONN_01X03
- added R10: 330, Resistors_SMD:R_0805, symbol R
- C1, C2, C3: footprint (none) -> Capacitors_SMD:C_0603
- D1: symbol LED -> LED-RESCUE-verseWriter
- P3: footprint (none) -> Connectors_JST:JST_XH_B04B-XH-A_04x2.50mm_Straight
- R1: renamed from R10; footprint Resistors_SMD:R_0805_HandSoldering -> Resistors_SMD:R_0805
- R11, R12: footprint Resistors_SMD:R_0805_HandSoldering -> Resistors_SMD:R_0805
- R13: renamed from R1; footprint Resistors_SMD:R_0805_HandSoldering -> Resistors_SMD:R_0805
- R2, R4, R6, R9: value 1k -> 330; footprint Resistors_SMD:R_0805_HandSoldering -> Resistors_SMD:R_0805
- R3, R5, R7: value 2k -> 330; footprint Resistors_SMD:R_0805_HandSoldering -> Resistors_SMD:R_0805
- R8: value 10 -> 330; footprint Resistors_SMD:R_0805_HandSoldering -> Resistors_SMD:R_0805
- SW1: footprint (none) -> Buttons_Switches_SMD:SW_SPST_KMR2
- Y1: footprint (none) -> Crystals:Crystal_HC18-U_Vertical
Connections:
- wire segments 191 -> 125
- no-connect marks 9 -> 6
Other:
- moved on the sheet: R1

Commit message: Finish
Parts:
- removed P3: Writer, Connectors_JST:JST_XH_B04B-XH-A_04x2.50mm_Straight, symbol CONN_01X04
- added C4: 100n, Capacitors_SMD:C_0603, symbol C
- added P2: FT-232R, Pin_Headers:Pin_Header_Straight_1x06_Pitch2.54mm, symbol CONN_01X06
- CON1: footprint (none) -> SparkFun-Footprints:SF-MICRO-SD
Connections:
- net GND: now also P2.1 (P1)
- net at IC1.29 ((PCINT14/~RESET~)PC6), R13.2, SW1.2: now also C4.1
- net at IC1.30 ((PCINT16/RXD)PD0): now also P2.4 (P4)
- net at IC1.31 ((PCINT17/TXD)PD1): now also P2.5 (P5)
- new net: C4.2, P2.6 (P6)
- no-connect marks 6 -> 8
Changed lines of the file:
@@
 $EndComp
 $Comp
-L CONN_01X04 P3
-U 1 1 58B9ACA9
-P 5400 4700
-F 0 "P3" H 5400 4950 50  0000 C CNN
-F 1 "Writer" V 5500 4700 50  0000 C CNN
-F 2 "Connectors_JST:JST_XH_B04B-XH-A_04x2.50mm_Straight" H 5400 4700 50  0001 C CNN
-F 3 "" H 5400 4700 50  0000 C CNN
-	1    5400 4700
-	1    0    0    -1
-$EndComp
-$Comp
-L VCC #PWR010
-U 1 1 58B9AF22
-P 5150 4500
-F 0 "#PWR010" H 5150 4350 50  0001 C CNN
-F 1 "VCC" H 5150 4650 50  0000 C CNN
-F 2 "" H 5150 4500 60  0000 C CNN
-F 3 "" H 5150 4500 60  0000 C CNN
-	1    5150 4500
-	1    0    0    -1
-$EndComp
-$Comp
-L GND #PWR011
+L GND #PWR010
 U 1 1 58B9B021
-P 5150 4900
-F 0 "#PWR011" H 5150 4650 50  0001 C CNN
-F 1 "GND" H 5150 4750 50  0000 C CNN
-F 2 "" H 5150 4900 60  0000 C CNN
-F 3 "" H 5150 4900 60  0000 C CNN
-	1    5150 4900
-	1    0    0    -1
-$EndComp
-Wire Wire Line
-	5200 4650 5050 4650
-Wire Wire Line
-	5050 4650 5050 3500
-Wire Wire Line
-	5000 3600 5000 4750
-Wire Wire Line
-	5000 4750 5200 4750
-Wire Wire Line
-	5200 4850 5150 4850
-Wire Wire Line
-	5150 4850 5150 4900
-Wire Wire Line
-	5200 4550 5150 4550
-Wire Wire Line
-	5150 4550 5150 4500
-$Comp
-L VCC #PWR012
+P 5650 5250
+F 0 "#PWR010" H 5650 5000 50  0001 C CNN
+F 1 "GND" H 5650 5100 50  0000 C CNN
+F 2 "" H 5650 5250 60  0000 C CNN
+F 3 "" H 5650 5250 60  0000 C CNN
+	1    5650 5250
+	0    1    1    0
+$EndComp
+Wire Wire Line
+	5050 3500 5050 5550
+Wire Wire Line
+	5000 3600 5000 5650
+$Comp
+L VCC #PWR011
 U 1 1 58BA7D46
 P 2050 1900
-F 0 "#PWR012" H 2050 1750 50  0001 C CNN
+F 0 "#PWR011" H 2050 1750 50  0001 C CNN
 F 1 "VCC" H 2050 2050 50  0000 C CNN
 F 2 "" H 2050 1900 50  0000 C CNN
@@
 $EndComp
 $Comp
-L GND #PWR013
+L GND #PWR012
 U 1 1 58BA7DD0
 P 2050 2300
-F 0 "#PWR013" H 2050 2050 50  0001 C CNN
+F 0 "#PWR012" H 2050 2050 50  0001 C CNN
 F 1 "GND" H 2050 2150 50  0000 C CNN
 F 2 "" H 2050 2300 50  0000 C CNN
@@
 	2350 1950 2350 1900
 $Comp
-L PWR_FLAG #FLG014
+L PWR_FLAG #FLG013
 U 1 1 58BA8296
 P 2350 1900
-F 0 "#FLG014" H 2350 1995 50  0001 C CNN
+F 0 "#FLG013" H 2350 1995 50  0001 C CNN
 F 1 "PWR_FLAG" H 2350 2080 50  0000 C CNN
 F 2 "" H 2350 1900 50  0000 C CNN
@@
 $EndComp
 $Comp
-L PWR_FLAG #FLG015
+L PWR_FLAG #FLG014
 U 1 1 58BA8359
 P 2350 2250
-F 0 "#FLG015" H 2350 2345 50  0001 C CNN
+F 0 "#FLG014" H 2350 2345 50  0001 C CNN
 F 1 "PWR_FLAG" H 2350 2430 50  0000 C CNN
 F 2 "" H 2350 2250 50  0000 C CNN
@@
 	4900 3350 4950 3350
 Wire Wire Line
-	4950 3350 4950 5250
+	4950 3350 4950 5750
 $Comp
 L LED-RESCUE-verseWriter D2
@@
 NoConn ~ 4900 3150
 $Comp
-L GND #PWR016
+L GND #PWR015
 U 1 1 58CDF12F
 P 8750 3050
-F 0 "#PWR016" H 8750 2800 50  0001 C CNN
+F 0 "#PWR015" H 8750 2800 50  0001 C CNN
 F 1 "GND" H 8750 2900 50  0000 C CNN
 F 2 "" H 8750 3050 60  0000 C CNN
@@
 Connection ~ 1500 3000
 $Comp
-L VCC #PWR017
+L VCC #PWR016
 U 1 1 58CF0CEC
 P 2200 3150
-F 0 "#PWR017" H 2200 3000 50  0001 C CNN
+F 0 "#PWR016" H 2200 3000 50  0001 C CNN
 F 1 "VCC" H 2200 3300 50  0000 C CNN
 F 2 "" H 2200 3150 50  0000 C CNN
@@
 $EndComp
 $Comp
-L GND #PWR018
+L GND #PWR017
 U 1 1 58CF0D4C
 P 1000 3550
-F 0 "#PWR018" H 1000 3300 50  0001 C CNN
+F 0 "#PWR017" H 1000 3300 50  0001 C CNN
 F 1 "GND" H 1000 3400 50  0000 C CNN
 F 2 "" H 1000 3550 50  0000 C CNN
@@
 $EndComp
 $Comp
-L VCC #PWR019
+L VCC #PWR018
 U 1 1 58CF63C6
 P 5300 3050
-F 0 "#PWR019" H 5300 2900 50  0001 C CNN
+F 0 "#PWR018" H 5300 2900 50  0001 C CNN
 F 1 "VCC" H 5300 3200 50  0000 C CNN
 F 2 "" H 5300 3050 50  0000 C CNN
@@
 F 0 "CON1" H 7000 5350 50  0000 C CNN
 F 1 "Micro_SD_Card" H 8300 5350 50  0000 R CNN
-F 2 "" H 8800 5050 50  0001 C CNN
+F 2 "SparkFun-Footprints:SF-MICRO-SD" H 8800 5050 50  0001 C CNN
 F 3 "" H 7650 4750 50  0000 C CNN
 	1    7650 4750
@@
 NoConn ~ 6750 4450
 $Comp
-L GND #PWR020
+L GND #PWR019
 U 1 1 58D03411
 P 8500 5400
-F 0 "#PWR020" H 8500 5150 50  0001 C CNN
+F 0 "#PWR019" H 8500 5150 50  0001 C CNN
 F 1 "GND" H 8500 5250 50  0000 C CNN
 F 2 "" H 8500 5400 60  0000 C CNN
@@
 Wire Wire Line
 	8500 5350 8500 5400
+$Comp
+L CONN_01X06 P2
+U 1 1 58D51686
+P 5850 5500
+F 0 "P2" H 5850 5850 50  0000 C CNN
+F 1 "FT-232R" V 5950 5500 50  0000 C CNN
+F 2 "Pin_Headers:Pin_Header_Straight_1x06_Pitch2.54mm" H 5850 5500 50  0001 C CNN
+F 3 "" H 5850 5500 50  0000 C CNN
+	1    5850 5500
+	1    0    0    -1
+$EndComp
+Wire Wire Line
+	5050 5550 5650 5550
+Wire Wire Line
+	5000 5650 5650 5650
+NoConn ~ 5650 5450
+$Comp
+L C C4
+U 1 1 58D53614
+P 5350 5750
+F 0 "C4" H 5375 5850 50  0000 L CNN
+F 1 "100n" H 5375 5650 50  0000 L CNN
+F 2 "Capacitors_SMD:C_0603" H 5388 5600 50  0001 C CNN
+F 3 "" H 5350 5750 50  0000 C CNN
+	1    5350 5750
+	0    -1   1    0
+$EndComp
+NoConn ~ 5650 5350
+Wire Wire Line
+	5650 5750 5500 5750
+Wire Wire Line
+	4950 5750 5200 5750
+Connection ~ 4950 5250
 $EndSCHEMATC

Commit message: Add AVR-ISP
Parts:
- added CON2: AVR-ISP-6, Pin_Headers:Pin_Header_Straight_2x03_Pitch2.54mm, symbol AVR-ISP-6
- added P3: IR, Pin_Headers:Pin_Header_Straight_1x03_Pitch2.54mm, symbol CONN_01X03
Connections:
- net GND: now also CON2.6, P3.2 (P2)
- net VCC: now also CON2.2, P3.1 (P1)
- net at C4.1, IC1.29 ((PCINT14/~RESET~)PC6), R13.2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: now also CON2.5
- net at CON1.3 (CMD), IC1.15 ((PCINT3/OC2A/MOSI)PB3): now also CON2.4
- net at IC1.16 ((PCINT4/MISO)PB4): now also CON1.7 (DAT0), CON2.1; no longer CON1.5 (CLK)
- net at IC1.17 ((PCINT5/SCK)PB5): now also CON1.5 (CLK), CON2.3; no longer CON1.7 (DAT0)
- net at IC1.27 ((PCINT12/SDA/ADC4)PC4): now also P3.3 (P3)
- no-connect marks 8 -> 7

Commit message: 微修正
Parts:
- removed CON2: AVR-ISP-6, Pin_Headers:Pin_Header_Straight_2x03_Pitch2.54mm, symbol AVR-ISP-6
- added P5: AVR-ISP, Pin_Headers:Pin_Header_Straight_1x05_Pitch2.54mm, symbol CONN_01X05
- CON1: footprint SparkFun-Footprints:SF-MICRO-SD -> conn-io:HIROSE-MICROSD-DM3AT-SF
- P3: footprint Pin_Headers:Pin_Header_Straight_1x03_Pitch2.54mm -> Connectors_JST:JST_PH_B3B-PH-SM4-TB_03x2.00mm_Straight
Connections:
- net GND: now also P5.5 (P5)
- net at C4.1, IC1.29 ((PCINT14/~RESET~)PC6), R13.2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: now also P5.4 (P4)
- net at CON1.3 (CMD), IC1.15 ((PCINT3/OC2A/MOSI)PB3): now also P5.3 (P3)
- net at CON1.7 (DAT0), IC1.16 ((PCINT4/MISO)PB4): now also P5.1 (P1)
- net at CON1.5 (CLK), IC1.17 ((PCINT5/SCK)PB5): now also P5.2 (P2)
Changed lines of the file:
@@
 F 0 "CON1" H 7000 5350 50  0000 C CNN
 F 1 "Micro_SD_Card" H 8300 5350 50  0000 R CNN
-F 2 "SparkFun-Footprints:SF-MICRO-SD" H 8800 5050 50  0001 C CNN
+F 2 "conn-io:HIROSE-MICROSD-DM3AT-SF" H 8800 5050 50  0001 C CNN
 F 3 "" H 7650 4750 50  0000 C CNN
 	1    7650 4750
@@
 NoConn ~ 5650 5350
 $Comp
-L AVR-ISP-6 CON2
-U 1 1 58D7FAA6
-P 7400 6050
-F 0 "CON2" H 7295 6290 50  0000 C CNN
-F 1 "AVR-ISP-6" H 7135 5820 50  0000 L BNN
-F 2 "Pin_Headers:Pin_Header_Straight_2x03_Pitch2.54mm" V 6880 6090 50  0001 C CNN
-F 3 "" H 7375 6050 50  0000 C CNN
-	1    7400 6050
-	1    0    0    -1
-$EndComp
-$Comp
 L GND #PWR020
 U 1 1 58D83BBB
-P 7800 6150
-F 0 "#PWR020" H 7800 5900 50  0001 C CNN
-F 1 "GND" H 7800 6000 50  0000 C CNN
-F 2 "" H 7800 6150 60  0000 C CNN
-F 3 "" H 7800 6150 60  0000 C CNN
-	1    7800 6150
-	0    -1   -1   0
-$EndComp
-$Comp
-L VCC #PWR021
-U 1 1 58D83C16
-P 7800 5950
-F 0 "#PWR021" H 7800 5800 50  0001 C CNN
-F 1 "VCC" H 7800 6100 50  0000 C CNN
-F 2 "" H 7800 5950 50  0000 C CNN
-F 3 "" H 7800 5950 50  0000 C CNN
-	1    7800 5950
+P 7300 6150
+F 0 "#PWR020" H 7300 5900 50  0001 C CNN
+F 1 "GND" H 7300 6000 50  0000 C CNN
+F 2 "" H 7300 6150 60  0000 C CNN
+F 3 "" H 7300 6150 60  0000 C CNN
+	1    7300 6150
 	0    1    1    0
 $EndComp
@@
 F 0 "P3" H 5700 6850 50  0000 C CNN
 F 1 "IR" V 5800 6650 50  0000 C CNN
-F 2 "Pin_Headers:Pin_Header_Straight_1x03_Pitch2.54mm" H 5700 6650 50  0001 C CNN
+F 2 "Connectors_JST:JST_PH_B3B-PH-SM4-TB_03x2.00mm_Straight" H 5700 6650 50  0001 C CNN
 F 3 "" H 5700 6650 50  0000 C CNN
 	1    5700 6650
@@
 	4900 3350 5050 3350
 Wire Wire Line
-	5050 3350 5050 6150
+	5050 3350 5050 6050
 Wire Wire Line
 	8450 850  8750 850
@@
 Connection ~ 5050 5250
 Wire Wire Line
-	7250 5950 6300 5950
-Wire Wire Line
-	6300 5950 6300 5050
+	6300 5050 6300 5750
 Connection ~ 6300 5050
 Wire Wire Line
-	7250 6050 6150 6050
-Wire Wire Line
-	6150 6050 6150 4850
+	6150 4850 6150 5850
 Connection ~ 6150 4850
-Wire Wire Line
-	5050 6150 7250 6150
 Connection ~ 5050 5750
 Wire Wire Line
-	7500 6050 7950 6050
-Wire Wire Line
-	7950 6050 7950 5700
-Wire Wire Line
-	7950 5700 6400 5700
-Wire Wire Line
-	6400 5700 6400 4650
+	6400 4650 6400 5950
 Connection ~ 6400 4650
 Wire Wire Line
-	7800 5950 7500 5950
-Wire Wire Line
-	7800 6150 7500 6150
-Wire Wire Line
 	6150 1900 4900 1900
 Wire Wire Line
@@
 	4950 3150 4900 3150
 $Comp
-L VCC #PWR022
+L VCC #PWR021
 U 1 1 58D92722
 P 5350 6550
-F 0 "#PWR022" H 5350 6400 50  0001 C CNN
+F 0 "#PWR021" H 5350 6400 50  0001 C CNN
 F 1 "VCC" H 5350 6700 50  0000 C CNN
 F 2 "" H 5350 6550 50  0000 C CNN
@@
 $EndComp
 $Comp
-L GND #PWR023
+L GND #PWR022
 U 1 1 58D927B2
 P 5500 6650
-F 0 "#PWR023" H 5500 6400 50  0001 C CNN
+F 0 "#PWR022" H 5500 6400 50  0001 C CNN
 F 1 "GND" H 5500 6500 50  0000 C CNN
 F 2 "" H 5500 6650 60  0000 C CNN
@@
 Wire Wire Line
 	4950 6750 5500 6750
+$Comp
+L CONN_01X05 P5
+U 1 1 58D95536
+P 7500 5950
+F 0 "P5" H 7500 6250 50  0000 C CNN
+F 1 "AVR-ISP" V 7600 5950 50  0000 C CNN
+F 2 "Pin_Headers:Pin_Header_Straight_1x05_Pitch2.54mm" H 7500 5950 50  0001 C CNN
+F 3 "" H 7500 5950 50  0000 C CNN
+	1    7500 5950
+	1    0    0    -1
+$EndComp
+Wire Wire Line
+	6300 5750 7300 5750
+Wire Wire Line
+	6150 5850 7300 5850
+Wire Wire Line
+	6400 5950 7300 5950
+Wire Wire Line
+	5050 6050 7300 6050
 $EndSCHEMATC

Commit message: 完成
Parts:
- P3: footprint Connectors_JST:JST_PH_B3B-PH-SM4-TB_03x2.00mm_Straight -> Pin_Headers:Pin_Header_Straight_1x03_Pitch2.54mm
Changed lines of the file:
@@
 F 0 "P3" H 5700 6850 50  0000 C CNN
 F 1 "IR" V 5800 6650 50  0000 C CNN
-F 2 "Connectors_JST:JST_PH_B3B-PH-SM4-TB_03x2.00mm_Straight" H 5700 6650 50  0001 C CNN
+F 2 "Pin_Headers:Pin_Header_Straight_1x03_Pitch2.54mm" H 5700 6650 50  0001 C CNN
 F 3 "" H 5700 6650 50  0000 C CNN
 	1    5700 6650
