File: circuit/verseWriter.kicad_pcb (KiCad board)
At the start: 2 copper layers, 20 x 120 mm, 38 parts, among them CON1 Micro_SD_Card, IC1 ATMEGA328P-A, P1 HOLE, P2 FT-232R, P4 SW, SW1 RESET, Y1 16M

Commit message: Add AVR-ISP
Parts:
- added AVR-ISP: AVR-ISP, Pin_Headers:Pin_Header_Straight_1x05_Pitch2.54mm, F.Cu at (192.5, 108.2)
- CON1: footprint SparkFun-Footprints:SF-MICRO-SD -> conn-io:HIROSE-MICROSD-DM3AT-SF
- moved CON1 5.78 mm to (175.4, 116.9)
Connections:
- IC1 pad 16: Net-(CON1-Pad5) -> Net-(CON1-Pad7)
- IC1 pad 17: Net-(CON1-Pad7) -> Net-(CON1-Pad5)
- IC1 pad 27: (no net) -> Net-(IC1-Pad27)
Routing:
- net GND: track 139.9 -> 193.6 mm, vias 4 -> 6
- net VCC: track 72.6 -> 111.6 mm, vias 4 -> 6
- net Net-(CON1-Pad3): track 25.1 -> 43.4 mm, vias 0 -> 2
- net Net-(CON1-Pad2): track 22.8 -> 30.2 mm
- net Net-(CON1-Pad5): track 24.9 -> 31.1 mm
- net Net-(C4-Pad1): track 35.8 -> 41.3 mm
- net (no net): track 2.00 -> 0.00 mm, vias 2 -> 0
- net Net-(CON1-Pad7): track 24.5 -> 26.5 mm, vias 0 -> 2
- net Net-(C2-Pad2): track 13.7 -> 15.7 mm
- net Net-(IC1-Pad25): track 44.1 -> 42.6 mm
- net Net-(C3-Pad2): track 10.4 -> 11.3 mm
- net Net-(IC1-Pad28): track 34.3 -> 34.8 mm, vias 0 -> 2

Commit message: 微修正
Parts:
- renumbered IC1 to ATMEGA38, P1 to HOLE, CON1 to MicroSD, P4 to ON-OFF, SW1 to RESET, P2 to Serial
Routing:
- net GND: track 193.6 -> 160.3 mm
- net (no net): vias 0 -> 2
Changed lines of the file:
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@@
     (links 78)
     (no_connects 0)
-    (area 174.899999 14.724999 213.564286 151.000001)
+    (area 173.599999 14.724999 213.564286 142.700001)
     (thickness 1.6)
     (drawings 9)
-    (tracks 451)
+    (tracks 455)
     (zones 0)
     (modules 39)
@@
     (47 F.CrtYd user)
     (48 B.Fab user)
-    (49 F.Fab user)
+    (49 F.Fab user hide)
   )
   (setup
@@
     (tags microsd)
     (clearance 0.254)
-    (fp_text reference CON1 (at 8.128 -17.653 360) (layer F.SilkS)
+    (fp_text reference MicroSD (at 8.11 -11.619 360) (layer F.SilkS)
       (effects (font (size 1 1) (thickness 0.18)) (justify right top))
     )
@@
     (tags "capacitor 0603")
     (attr smd)
-    (fp_text reference C2 (at 0 -1.5 180) (layer F.SilkS)
+    (fp_text reference C2 (at 0 1.575 180) (layer F.SilkS)
       (effects (font (size 1 1) (thickness 0.15)))
     )
@@
     (tags "QFP 0.8")
     (attr smd)
-    (fp_text reference IC1 (at 0 -6.05 270) (layer F.SilkS)
+    (fp_text reference ATMEGA38 (at 6.75 0 360) (layer F.SilkS)
       (effects (font (size 1 1) (thickness 0.15)))
     )
@@
     (descr "Through hole straight pin header, 1x03, 2.54mm pitch, single row")
     (tags "Through hole pin header THT 1x03 2.54mm single row")
-    (fp_text reference P1 (at 0 -2.39 180) (layer F.SilkS)
+    (fp_text reference HOLE (at -3 1.5 270) (layer F.SilkS)
       (effects (font (size 1 1) (thickness 0.15)))
     )
@@
     (descr "Through hole straight pin header, 1x03, 2.54mm pitch, single row")
     (tags "Through hole pin header THT 1x03 2.54mm single row")
-    (fp_text reference P4 (at 0 -2.39 180) (layer F.SilkS)
+    (fp_text reference ON-OFF (at -3 2 270) (layer F.SilkS)
       (effects (font (size 1 1) (thickness 0.15)))
     )
@@
     (tags "tactile switch kmr2")
     (attr smd)
-    (fp_text reference SW1 (at 0 -2.45 270) (layer F.SilkS)
+    (fp_text reference RESET (at -5 -1 270) (layer F.SilkS)
       (effects (font (size 1 1) (thickness 0.15)))
     )
@@
     (descr "Through hole straight pin header, 1x06, 2.54mm pitch, single row")
     (tags "Through hole pin header THT 1x06 2.54mm single row")
-    (fp_text reference P2 (at 0 -2.33) (layer F.SilkS)
+    (fp_text reference Serial (at 0 -4.13 90) (layer F.SilkS)
       (effects (font (size 1 1) (thickness 0.15)))
     )
@@
     (arrow2b (pts (xy 205 135) (xy 204.413579 133.873496)))
   )
+  (via (at 193 75) (size 3.2) (drill 3) (layers F.Cu B.Cu) (net 0))
+  (via (at 177 75) (size 3.2) (drill 3) (layers F.Cu B.Cu) (net 0))
   (segment (start 180.4 132) (end 185 132) (width 1) (layer B.Cu) (net 1))
   (segment (start 178 132) (end 180.4 132) (width 1) (layer B.Cu) (net 1))
@@
   (segment (start 185 87.2) (end 185 85.785787) (width 1) (layer B.Cu) (net 2))
   (segment (start 184.524969 64.289244) (end 185 63.814213) (width 1) (layer B.Cu) (net 2))
+  (segment (start 191.356999 100.643001) (end 191 101) (width 0.25) (layer B.Cu) (net 3))
+  (segment (start 192.532 98.044) (end 191.356999 99.219001) (width 0.25) (layer B.Cu) (net 3))
+  (segment (start 191.356999 99.219001) (end 191.356999 100.643001) (width 0.25) (layer B.Cu) (net 3))
   (segment (start 191 115) (end 191 114) (width 0.25) (layer B.Cu) (net 3))
   (segment (start 191.41 114.59) (end 191 115) (width 0.25) (layer F.Cu) (net 3))
@@
   (segment (start 180.5 92.625) (end 180.875 93) (width 0.25) (layer F.Cu) (net 3))
   (segment (start 194.175001 94.824999) (end 194.175001 86) (width 0.25) (layer B.Cu) (net 3))
-  (segment (start 194.175001 86) (end 194.175001 49.175001) (width 0.25) (layer B.Cu) (net 3))
   (segment (start 194 81) (end 194 85.824999) (width 0.25) (layer B.Cu) (net 3))
   (segment (start 194 85.824999) (end 194.175001 86) (width 0.25) (layer B.Cu) (net 3))

Commit message: 完成
Parts:
- added P3: IR, Pin_Headers:Pin_Header_Straight_1x03_Pitch2.54mm, B.Cu at (193.0, 132.5)
Routing:
- net Net-(IC1-Pad27): track 0.00 -> 32.3 mm, vias 0 -> 2
- net VCC: track 111.6 -> 114.6 mm, vias 6 -> 4
- net GND: track 160.3 -> 159.1 mm
- net Net-(IC1-Pad28): track 34.8 -> 33.7 mm
- net Net-(IC1-Pad26): track 26.2 -> 26.7 mm

Commit message: PCBgogo発注
Parts:
- added ATMEGA38: ATMEGA328P-A, Housings_QFP:TQFP-32_7x7mm_Pitch0.8mm, F.Cu at (225.0, 98.2)
- added ATMEGA38: ATMEGA328P-A, Housings_QFP:TQFP-32_7x7mm_Pitch0.8mm, F.Cu at (205.0, 98.2)
- added AVR-ISP: AVR-ISP, Pin_Headers:Pin_Header_Straight_1x05_Pitch2.54mm, F.Cu at (232.5, 108.2)
- added AVR-ISP: AVR-ISP, Pin_Headers:Pin_Header_Straight_1x05_Pitch2.54mm, F.Cu at (212.5, 108.2)
- added BT1: AAA, .pretty:AAA, B.Cu at (225.0, 109.6)
- added BT1: AAA, .pretty:AAA, B.Cu at (205.0, 109.6)
- added BT2: AAA, .pretty:AAA, B.Cu at (225.0, 40.0)
- added BT2: AAA, .pretty:AAA, B.Cu at (205.0, 40.0)
- added C1: C, Capacitors_SMD:C_0603, F.Cu at (226.2, 92.0)
- added C1: C, Capacitors_SMD:C_0603, F.Cu at (206.2, 92.0)
- added C2: 22p, Capacitors_SMD:C_0603, F.Cu at (223.8, 92.1)
- added C2: 22p, Capacitors_SMD:C_0603, F.Cu at (203.8, 92.1)
- added C3: 22p, Capacitors_SMD:C_0603, F.Cu at (221.2, 92.0)
- added C3: 22p, Capacitors_SMD:C_0603, F.Cu at (201.2, 92.0)
- added C4: 100n, Capacitors_SMD:C_0603, F.Cu at (233.0, 68.8)
- added C4: 100n, Capacitors_SMD:C_0603, F.Cu at (213.0, 68.8)
- added D1: LED, LEDs:LED_0805, F.Cu at (225.0, 20.0)
- added D1: LED, LEDs:LED_0805, F.Cu at (205.0, 20.0)
- added D10: LED, LEDs:LED_0805, F.Cu at (225.0, 65.0)
- added D10: LED, LEDs:LED_0805, F.Cu at (205.0, 65.0)
- added D11: LED, LEDs:LED_0805, F.Cu at (225.0, 70.0)
- added D11: LED, LEDs:LED_0805, F.Cu at (205.0, 70.0)
- added D12: LED, LEDs:LED_0805, F.Cu at (225.0, 75.0)
- added D12: LED, LEDs:LED_0805, F.Cu at (205.0, 75.0)
- added D2: LED, LEDs:LED_0805, F.Cu at (225.0, 25.0)
- added D2: LED, LEDs:LED_0805, F.Cu at (205.0, 25.0)
- added D3: LED, LEDs:LED_0805, F.Cu at (225.0, 30.0)
- added D3: LED, LEDs:LED_0805, F.Cu at (205.0, 30.0)
- added D4: LED, LEDs:LED_0805, F.Cu at (225.0, 35.0)
- added D4: LED, LEDs:LED_0805, F.Cu at (205.0, 35.0)
- added D5: LED, LEDs:LED_0805, F.Cu at (225.0, 40.0)
- added D5: LED, LEDs:LED_0805, F.Cu at (205.0, 40.0)
- added D6: LED, LEDs:LED_0805, F.Cu at (225.0, 45.0)
- added D6: LED, LEDs:LED_0805, F.Cu at (205.0, 45.0)
- added D7: LED, LEDs:LED_0805, F.Cu at (225.0, 50.0)
- added D7: LED, LEDs:LED_0805, F.Cu at (205.0, 50.0)
- added D8: LED, LEDs:LED_0805, F.Cu at (225.0, 55.0)
- added D8: LED, LEDs:LED_0805, F.Cu at (205.0, 55.0)
- added D9: LED, LEDs:LED_0805, F.Cu at (225.0, 60.0)
- added D9: LED, LEDs:LED_0805, F.Cu at (205.0, 60.0)
- added HOLE: HOLE, Pin_Headers:Pin_Header_Straight_1x03_Pitch2.54mm, F.Cu at (230.0, 132.5)
- added HOLE: HOLE, Pin_Headers:Pin_Header_Straight_1x03_Pitch2.54mm, F.Cu at (210.0, 132.5)
- added MicroSD: Micro_SD_Card, conn-io:HIROSE-MICROSD-DM3AT-SF, F.Cu at (215.4, 116.9)
- added MicroSD: Micro_SD_Card, conn-io:HIROSE-MICROSD-DM3AT-SF, F.Cu at (195.4, 116.9)
- added ON-OFF: SW, Pin_Headers:Pin_Header_Straight_1x03_Pitch2.54mm, F.Cu at (218.0, 132.0)
- added ON-OFF: SW, Pin_Headers:Pin_Header_Straight_1x03_Pitch2.54mm, F.Cu at (198.0, 132.0)
- added P3: IR, Pin_Headers:Pin_Header_Straight_1x03_Pitch2.54mm, B.Cu at (233.0, 132.5)
- added P3: IR, Pin_Headers:Pin_Header_Straight_1x03_Pitch2.54mm, B.Cu at (213.0, 132.5)
- added R1: 330, Resistors_SMD:R_0805, F.Cu at (228.8, 20.0)
- added R1: 330, Resistors_SMD:R_0805, F.Cu at (208.8, 20.0)
- added R10: 330, Resistors_SMD:R_0805, F.Cu at (228.0, 66.0)
- added R10: 330, Resistors_SMD:R_0805, F.Cu at (208.0, 66.0)
- added R11: 330, Resistors_SMD:R_0805, F.Cu at (228.0, 71.0)
- added R11: 330, Resistors_SMD:R_0805, F.Cu at (208.0, 71.0)
- added R12: 330, Resistors_SMD:R_0805, F.Cu at (228.0, 76.0)
- added R12: 330, Resistors_SMD:R_0805, F.Cu at (208.0, 76.0)
- added R13: 1k, Resistors_SMD:R_0805, F.Cu at (232.9, 94.0)
- added R13: 1k, Resistors_SMD:R_0805, F.Cu at (212.9, 94.0)
- added R2: 330, Resistors_SMD:R_0805, F.Cu at (228.8, 25.0)
- added R2: 330, Resistors_SMD:R_0805, F.Cu at (208.8, 25.0)
- added R3: 330, Resistors_SMD:R_0805, F.Cu at (228.8, 30.0)
- added R3: 330, Resistors_SMD:R_0805, F.Cu at (208.8, 30.0)
- added R4: 330, Resistors_SMD:R_0805, F.Cu at (228.8, 35.0)
- added R4: 330, Resistors_SMD:R_0805, F.Cu at (208.8, 35.0)
- added R5: 330, Resistors_SMD:R_0805, F.Cu at (228.8, 40.0)
- added R5: 330, Resistors_SMD:R_0805, F.Cu at (208.8, 40.0)
- added R6: 330, Resistors_SMD:R_0805, F.Cu at (228.8, 45.0)
- added R6: 330, Resistors_SMD:R_0805, F.Cu at (208.8, 45.0)
- added R7: 330, Resistors_SMD:R_0805, F.Cu at (228.0, 51.0)
- added R7: 330, Resistors_SMD:R_0805, F.Cu at (208.0, 51.0)
- added R8: 330, Resistors_SMD:R_0805, F.Cu at (228.0, 56.0)
- added R8: 330, Resistors_SMD:R_0805, F.Cu at (208.0, 56.0)
- added R9: 330, Resistors_SMD:R_0805, F.Cu at (228.0, 61.0)
- added R9: 330, Resistors_SMD:R_0805, F.Cu at (208.0, 61.0)
- added RESET: RESET, Buttons_Switches_SMD:SW_SPST_KMR2, F.Cu at (233.0, 89.0)
- added RESET: RESET, Buttons_Switches_SMD:SW_SPST_KMR2, F.Cu at (213.0, 89.0)
- added Serial: FT-232R, Pin_Headers:Pin_Header_Straight_1x06_Pitch2.54mm, F.Cu at (233.0, 52.4)
- added Serial: FT-232R, Pin_Headers:Pin_Header_Straight_1x06_Pitch2.54mm, F.Cu at (213.0, 52.4)
- added Y1: 16M, Crystals:Crystal_HC18-U_Vertical, F.Cu at (227.5, 83.0)
- added Y1: 16M, Crystals:Crystal_HC18-U_Vertical, F.Cu at (207.5, 83.0)
Routing:
- net GND: track 159.1 -> 477.2 mm, vias 6 -> 18
- net VCC: track 114.6 -> 343.7 mm, vias 4 -> 12
- net Net-(IC1-Pad13): track 111.0 -> 332.9 mm
- net Net-(IC1-Pad12): track 92.3 -> 276.9 mm
- net Net-(IC1-Pad32): track 68.1 -> 204.4 mm, vias 2 -> 6
- net Net-(IC1-Pad9): track 62.5 -> 187.6 mm
- net Net-(IC1-Pad1): track 61.7 -> 185.1 mm
- net Net-(IC1-Pad2): track 57.0 -> 171.1 mm
- net Net-(IC1-Pad10): track 56.4 -> 169.1 mm, vias 2 -> 6
- net Net-(IC1-Pad11): track 53.9 -> 161.7 mm, vias 2 -> 6
- net Net-(IC1-Pad23): track 47.1 -> 141.3 mm, vias 2 -> 6
- net Net-(CON1-Pad3): track 43.3 -> 129.9 mm, vias 2 -> 6
- net Net-(IC1-Pad25): track 42.6 -> 127.8 mm, vias 2 -> 6
- net Net-(IC1-Pad24): track 42.1 -> 126.2 mm, vias 2 -> 6
- net Net-(IC1-Pad30): track 41.8 -> 125.5 mm, vias 1 -> 3
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Other:
- board size 20 x 120 mm -> 60 x 120 mm
- board text added: "Verse writer 2017.04.01 JP3CYC"
